Commit message: Testing various methods to get trajectory optimisation working

File: sliding_double_pendulum.urdf (robot description, URDF)
Before this commit: robot sliding_pendulum, 3 links, 3 joints
Links:
- link arm: mass 0.25 -> 0.187; geometry visual cylinder length=0.1645 radius=0.01; visual sphere radius=.015
- link forearm: mass 0.25 -> 0.132; geometry visual cylinder length=0.133 radius=0.01; visual sphere radius=0.015
- link slider: mass 1 -> 0.5; geometry visual box size=0.05 0.05 0.05
Joints:
- joint elbow: origin xyz=0 0 -0.5 -> xyz=0 0 -0.1645
