Commit message: LQR upright balancing working with single pendulum! Pendulum is oscillating very slowly, which I think is massively to do with friction

File: simulation/single_pendulum/single_pendulum.urdf (robot description, URDF)
Before this commit: robot sliding_pendulum, 2 links, 2 joints
Links:
- link slider: mass 0.5 -> 0.03
Joints:
- joint shoulder: axis 0 1 0 -> 0 -1 0
- joint slider_joint: axis 1 0 0 -> -1 0 0
